File: kicad/80bus.kicad_pcb (KiCad board)
At the start: 2 copper layers, 203.2 x 203.2 mm, 51 parts, among them J1 Conn_01x80NasBus, J2 Conn_02x25, J3 Power, Q1 2N3904, Q2 2N3904, SW1 SW_DIP_x08, U1 7406, U2 74LS74, U3 74LS32, U4 74LS244, U5 74LS244, U6 74LS244, U7 74LS138, U8 74LS32

Commit message: Fixing prototype issues
Parts:
- Q1, Q2: value 2N3904 -> 2N3906
- moved Q2 31.2 mm to (164.0, 58.0)
- moved Q1 31.2 mm to (164.2, 89.2)
- moved D2 27.1 mm to (168.6, 141.9), turned to 0 degrees
- moved R3 23.2 mm to (150.0, 133.6)
- moved TP1 17.4 mm to (173.0, 48.0)
- moved R4 4.50 mm to (171.1, 124.6)
- moved D4 2.97 mm to (177.2, 89.1), turned to 180 degrees
- moved D3 2.84 mm to (177.0, 58.0), turned to 180 degrees
- moved R8 0.72 mm to (163.5, 72.8)
- moved R12 0.72 mm to (163.5, 79.1)
- moved R9 0.72 mm to (163.4, 66.3)
Connections:
- D2 pad 2: VCC -> Net-(D2-A)
- J2 pad 45: Net-(J2-Pin_45) -> Net-(D2-K)
- Q1 pad 1: GND -> VCC
- Q1 pad 3: Net-(D3-K) -> Net-(D4-A)
- Q2 pad 1: GND -> VCC
- Q2 pad 3: Net-(D4-K) -> Net-(D3-A)
- R12 pad 1: VCC -> Net-(D4-K)
- R12 pad 2: Net-(D4-A) -> GND
- R4 pad 1: Net-(D2-K) -> VCC
- R4 pad 2: Net-(J2-Pin_45) -> Net-(D2-A)
- R6 pad 1: Net-(Q1-B) -> Net-(Q2-B)
- R8 pad 1: VCC -> Net-(D3-K)
- R8 pad 2: Net-(D3-A) -> GND
- R9 pad 1: Net-(Q2-B) -> Net-(Q1-B)
Routing:
- net Net-(J2-Pin_45): track 60.0 -> 0.00 mm, vias 1 -> 0
- net VCC: track 879.6 -> 921.8 mm, vias 3 -> 4
- net Net-(D2-K): track 10.3 -> 49.8 mm, vias 0 -> 1
- net Net-(J2-Pin_46): track 56.0 -> 78.0 mm, vias 0 -> 1
- net Net-(Q2-B): track 23.4 -> 42.8 mm
- net GND: track 969.7 -> 952.6 mm
- net Net-(D3-K): track 5.25 -> 22.1 mm
- net Net-(Q1-B): track 41.5 -> 26.2 mm
- net Net-(D4-K): track 5.18 -> 20.0 mm
- net Net-(D3-A): track 17.3 -> 5.41 mm
- net Net-(D2-A): track 0.00 -> 4.66 mm
- net Net-(D4-A): track 9.52 -> 5.40 mm
- net ~{IO_RD_ENABLE}: track 180.8 -> 179.0 mm
- net ~{BRESET}: track 214.4 -> 212.6 mm
- net Net-(J2-Pin_44): track 63.1 -> 61.3 mm
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Other:
- board text added: "+5V GND GND NC"
- board text added: "CF Timing Logic based on the circuit improvements by Tadeuzd Pycio http://www.vtsys.pl/interface-compact-flash"
- board text added: "Errata - Update CF connector footprint - Switch R/W Indicator Polarity"
- board text added: "Version 1.0.0 30e0750d-673c-4cc3-93fc-37be21742309"
- board text removed: "70d8a111-c327-4c3c-9c1b-054a19be2438"
- board text removed: "Errata - Add power connector - Swap to 50 pin CF connector"
- board text removed: "Version 0.0.2"

Commit message: Documentation
Parts:
- added R10: 10K, Resistor_THT:R_Axial_DIN0309_L9.0mm_D3.2mm_P12.70mm_Horizontal, F.Cu at (152.9, 74.7)
- added R11: 10K, Resistor_THT:R_Axial_DIN0309_L9.0mm_D3.2mm_P12.70mm_Horizontal, F.Cu at (152.9, 72.0)
Routing:
- net Net-(Q1-B): track 26.2 -> 45.3 mm
- net Net-(Q2-B): track 42.8 -> 61.3 mm
- net VCC: track 921.8 -> 929.7 mm
Other:
- board text added: "Errata - Add 10K pull up's to hard switch Q1, Q2"
- board text added: "Version 1.1 3cf8a701-0647-4ec0-a81e-45ad84dc77b7"
- board text removed: "Errata - Update CF connector footprint - Switch R/W Indicator Polarity"
- board text removed: "Version 1.0.0 30e0750d-673c-4cc3-93fc-37be21742309"

Commit message: Minor tweaks
Parts:
- added H1: Mount, TestPoint:TestPoint_Plated_Hole_D3.0mm, F.Cu at (169.5, 156.0)
- added H2: Mount, TestPoint:TestPoint_Plated_Hole_D3.0mm, F.Cu at (147.9, 156.0)
- added H3: Mount, TestPoint:TestPoint_Plated_Hole_D3.0mm, F.Cu at (147.9, 198.7)
- added H4: Mount, TestPoint:TestPoint_Plated_Hole_D3.0mm, F.Cu at (169.5, 198.7)
Routing:
- net ~{BRESET}: track 212.6 -> 217.6 mm
- net Net-(D2-K): track 49.8 -> 53.0 mm
- net ~{IO_RD_ENABLE}: track 179.0 -> 176.0 mm
- net Net-(J2-Pin_44): track 61.3 -> 62.9 mm
- net Net-(J2-Pin_46): track 78.0 -> 79.5 mm
- net ~{IO_WR_ENABLE}: track 298.5 -> 297.6 mm
Other:
- board text added: "Errata - Add 10K pull up's to hard switch Q1, Q2 - Support mount holes"
- board text added: "Things remembered in immortal minds"
- board text removed: "Errata - Add 10K pull up's to hard switch Q1, Q2"

Commit message: Docs and Kicad 9
Parts:
- added G001: LOGO, 80bus:qr code, B.Cu at (130.4, 169.9)
Other:
- board text added: "CS-005"
- board text added: "Documentation -->"
- board text added: "Version 1.2 / Kicad 9 659c61d7-5ee0-41bc-b8b7-7127bb9a5451"
- board text removed: "Version 1.1 3cf8a701-0647-4ec0-a81e-45ad84dc77b7"
