File: kicad/80bus.kicad_sch (KiCad schematic)
At the start: 50 parts, among them J1 Conn_01x80NasBus, J2 Conn_02x25, J3 Power, Q1 2N3904, Q2 2N3904, SW1 SW_DIP_x08, U1 7406, U2 74LS74, U3 74LS32, U4 74LS244, U5 74LS244, U6 74LS244, U7 74LS138, U8 74LS32

Commit message: Fixing prototype issues
Parts:
- removed Q1, Q2: 2N3904, Package_TO_SOT_THT:TO-92_Inline_Wide, symbol Transistor_BJT:2N3904
- added Q1, Q2: 2N3906, Package_TO_SOT_THT:TO-92_Inline_Wide, symbol Transistor_BJT:2N3906
Connections:
- net GND: now also R12.2, R8.2
- net VCC: now also R4.1, Q1.1 (E), Q2.1 (E); no longer D2.2 (A), R12.1, R8.1
- net at D2.1 (K): now also J2.45 (Pin_45); no longer R4.1
- net at R4.2: now also D2.2 (A); no longer J2.45 (Pin_45)
- net at R6.1: now also Q2.2 (B)
- net at D3.1 (K): now also R8.1
- net at D4.1 (K): now also R12.1
- net at D4.2 (A): now also Q1.3 (C); no longer R12.2
- net at R9.1: now also Q1.2 (B)
- net at D3.2 (A): now also Q2.3 (C); no longer R8.2
Other:
- moved on the sheet: D2, D3, D4, R12, R8

Commit message: Documentation
Parts:
- added R10, R11: 10K, Resistor_THT:R_Axial_DIN0309_L9.0mm_D3.2mm_P12.70mm_Horizontal, symbol Device:R
Connections:
- net VCC: now also R10.1, R11.1
- net at Q1.2 (B), R9.1: now also R10.2
- net at Q2.2 (B), R6.1: now also R11.2
Changed lines of the file:
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@@
   (title_block
     (title "80 Bus Compact Flash Card")
-    (date "2023-10-08")
-    (rev "1.0.0")
+    (date "2023-11-02")
+    (rev "1.1")
   )
   (junction (at 139.7 266.7) (diameter 0) (color 0 0 0 0)
@@
   (junction (at 105.41 266.7) (diameter 0) (color 0 0 0 0)
   )
+  (junction (at 364.49 233.68) (diameter 0) (color 0 0 0 0)
+  )
   (junction (at 276.86 226.06) (diameter 0) (color 0 0 0 0)
   )
@@
   (junction (at 279.4 71.12) (diameter 0) (color 0 0 0 0)
   )
+  (junction (at 345.44 156.21) (diameter 0) (color 0 0 0 0)
+  )
   (junction (at 313.69 33.02) (diameter 0) (color 0 0 0 0)
   )
@@
   (junction (at 71.12 240.03) (diameter 0) (color 0 0 0 0)
   )
+  (junction (at 335.28 167.64) (diameter 0) (color 0 0 0 0)
+  )
   (junction (at 355.6 78.74) (diameter 0) (color 0 0 0 0)
   )
@@
   (junction (at 50.8 220.98) (diameter 0) (color 0 0 0 0)
   )
+  (junction (at 373.38 223.52) (diameter 0) (color 0 0 0 0)
+  )
   (junction (at 254 154.94) (diameter 0) (color 0 0 0 0)
   )
@@
     (stroke (width 0) (type default))
   )
+  (wire (pts (xy 335.28 165.1) (xy 335.28 167.64))
+    (stroke (width 0) (type default))
+  )
   (wire (pts (xy 194.31 68.58) (xy 194.31 63.5))
     (stroke (width 0) (type default))
@@
     (stroke (width 0) (type default))
   )
-  (wire (pts (xy 345.44 154.94) (xy 345.44 162.56))
+  (wire (pts (xy 345.44 154.94) (xy 345.44 156.21))
     (stroke (width 0) (type default))
   )
@@
     (stroke (width 0) (type default))
   )
+  (wire (pts (xy 364.49 223.52) (xy 373.38 223.52))
+    (stroke (width 0) (type default))
+  )
   (wire (pts (xy 276.86 218.44) (xy 295.91 218.44))
     (stroke (width 0) (type default))
@@
     (stroke (width 0) (type default))
   )
-  (wire (pts (xy 326.39 167.64) (xy 337.82 167.64))
+  (wire (pts (xy 326.39 167.64) (xy 335.28 167.64))
     (stroke (width 0) (type default))
   )
@@
     (stroke (width 0) (type default))
   )
-  (wire (pts (xy 354.33 233.68) (xy 365.76 233.68))
+  (wire (pts (xy 354.33 233.68) (xy 364.49 233.68))
     (stroke (width 0) (type default))
   )
@@
     (stroke (width 0) (type default))
   )
+  (wire (pts (xy 345.44 156.21) (xy 345.44 162.56))
+    (stroke (width 0) (type default))
+  )
   (wire (pts (xy 276.86 218.44) (xy 267.97 218.44))
     (stroke (width 0) (type default))
@@
     (stroke (width 0) (type default))
   )
+  (wire (pts (xy 335.28 156.21) (xy 345.44 156.21))
+    (stroke (width 0) (type default))
+  )
   (wire (pts (xy 219.71 231.14) (xy 203.2 231.14))
     (stroke (width 0) (type default))
@@
     (stroke (width 0) (type default))
   )
+  (wire (pts (xy 335.28 157.48) (xy 335.28 156.21))
+    (stroke (width 0) (type default))
+  )
   (wire (pts (xy 104.14 129.54) (xy 106.68 129.54))
     (stroke (width 0) (type default))
@@
     (stroke (width 0) (type default))
   )
+  (wire (pts (xy 335.28 167.64) (xy 337.82 167.64))
+    (stroke (width 0) (type default))
+  )
   (wire (pts (xy 292.1 58.42) (xy 304.8 58.42))
     (stroke (width 0) (type default))
@@
     (stroke (width 0) (type default))
   )
+  (wire (pts (xy 364.49 233.68) (xy 365.76 233.68))
+    (stroke (width 0) (type default))
+  )
   (wire (pts (xy 276.86 236.22) (xy 276.86 233.68))
     (stroke (width 0) (type default))
@@
     (stroke (width 0) (type default))
   )
+  (wire (pts (xy 373.38 223.52) (xy 373.38 228.6))
+    (stroke (width 0) (type default))
+  )
   (wire (pts (xy 279.4 91.44) (xy 279.4 88.9))
     (stroke (width 0) (type default))
@@
     (stroke (width 0) (type default))
   )
+  (wire (pts (xy 364.49 231.14) (xy 364.49 233.68))
+    (stroke (width 0) (type default))
+  )
   (wire (pts (xy 106.68 104.14) (xy 104.14 104.14))
     (stroke (width 0) (type default))
@@
     (stroke (width 0) (type default))
   )
-  (wire (pts (xy 373.38 220.98) (xy 373.38 228.6))
+  (wire (pts (xy 373.38 220.98) (xy 373.38 223.52))
     (stroke (width 0) (type default))
   )
@@
     )
   )
+  (symbol (lib_id "Device:R") (at 335.28 161.29 0) (unit 1)
+    (in_bom yes) (on_board yes) (dnp no) (fields_autoplaced)
+    (property "Reference" "R11" (at 337.82 160.02 0)
+      (effects (font (size 1.27 1.27)) (justify left))
+    )
+    (property "Value" "10K" (at 337.82 162.56 0)
+      (effects (font (size 1.27 1.27)) (justify left))
+    )
+    (property "Footprint" "Resistor_THT:R_Axial_DIN0309_L9.0mm_D3.2mm_P12.70mm_Horizontal" (at 333.502 161.29 90)
+      (effects (font (size 1.27 1.27)) hide)
+    )
+    (property "Datasheet" "~" (at 335.28 161.29 0)
+      (effects (font (size 1.27 1.27)) hide)
+    )
+    (pin "1")
+    (pin "2")
+    (instances
+      (project "80bus"
+        (path "/c5a86bac-f144-45ed-8f39-1fb354fa8f6d"
+          (reference "R11") (unit 1)
+        )
+      )
+    )
+  )
   (symbol (lib_id "Device:LED") (at 322.58 63.5 0) (unit 1)
     (in_bom yes) (on_board yes) (dnp no)
@@
         )
       )
+    )
+  )
+  (symbol (lib_id "Device:R") (at 364.49 227.33 0) (unit 1)
+    (in_bom yes) (on_board yes) (dnp no) (fields_autoplaced)
+    (property "Reference" "R10" (at 367.03 226.06 0)
+      (effects (font (size 1.27 1.27)) (justify left))
+    )
+    (property "Value" "10K" (at 367.03 228.6 0)
+      (effects (font (size 1.27 1.27)) (justify left))
+    )
+    (property "Footprint" "Resistor_THT:R_Axial_DIN0309_L9.0mm_D3.2mm_P12.70mm_Horizontal" (at 362.712 227.33 90)
+      (effects (font (size 1.27 1.27)) hide)
+    )
+    (property "Datasheet" "~" (at 364.49 227.33 0)
+      (effects (font (size 1.27 1.27)) hide)
+    )
+    (pin "1")
+    (pin "2")
+    (instances
+      (project "80bus"
+        (path "/c5a86bac-f144-45ed-8f39-1fb354fa8f6d"
+          (reference "R10") (unit 1)
+        )
+      )

Commit message: Minor tweaks
Parts:
- added H1, H2, H3, H4: Mount, TestPoint:TestPoint_Plated_Hole_D3.0mm, symbol Mechanical:MountingHole
Changed lines of the file:
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@@
   (title_block
     (title "80 Bus Compact Flash Card")
-    (date "2023-11-02")
+    (date "2023-11-04")
     (rev "1.1")
   )
@@
     )
   )
+  (symbol (lib_id "Mechanical:MountingHole") (at 374.65 59.69 0) (unit 1)
+    (in_bom yes) (on_board yes) (dnp no) (fields_autoplaced)
+    (property "Reference" "H1" (at 377.19 58.42 0)
+      (effects (font (size 1.27 1.27)) (justify left))
+    )
+    (property "Value" "Mount" (at 377.19 60.96 0)
+      (effects (font (size 1.27 1.27)) (justify left))
+    )
+    (property "Footprint" "TestPoint:TestPoint_Plated_Hole_D3.0mm" (at 374.65 59.69 0)
+      (effects (font (size 1.27 1.27)) hide)
+    )
+    (property "Datasheet" "~" (at 374.65 59.69 0)
+      (effects (font (size 1.27 1.27)) hide)
+    )
+    (instances
+      (project "80bus"
+        (path "/c5a86bac-f144-45ed-8f39-1fb354fa8f6d"
+          (reference "H1") (unit 1)
+        )
+      )
+    )
+  )
   (symbol (lib_id "power:VCC") (at 345.44 96.52 180) (unit 1)
     (in_bom yes) (on_board yes) (dnp no) (fields_autoplaced)
@@
     )
   )
+  (symbol (lib_id "Mechanical:MountingHole") (at 374.65 72.39 0) (unit 1)
+    (in_bom yes) (on_board yes) (dnp no) (fields_autoplaced)
+    (property "Reference" "H3" (at 377.19 71.12 0)
+      (effects (font (size 1.27 1.27)) (justify left))
+    )
+    (property "Value" "Mount" (at 377.19 73.66 0)
+      (effects (font (size 1.27 1.27)) (justify left))
+    )
+    (property "Footprint" "TestPoint:TestPoint_Plated_Hole_D3.0mm" (at 374.65 72.39 0)
+      (effects (font (size 1.27 1.27)) hide)
+    )
+    (property "Datasheet" "~" (at 374.65 72.39 0)
+      (effects (font (size 1.27 1.27)) hide)
+    )
+    (instances
+      (project "80bus"
+        (path "/c5a86bac-f144-45ed-8f39-1fb354fa8f6d"
+          (reference "H3") (unit 1)
+        )
+      )
+    )
+  )
   (symbol (lib_id "74xx:74LS32") (at 38.1 257.81 90) (unit 5)
     (in_bom yes) (on_board yes) (dnp no) (fields_autoplaced)
@@
     )
   )
+  (symbol (lib_id "Mechanical:MountingHole") (at 374.65 66.04 0) (unit 1)
+    (in_bom yes) (on_board yes) (dnp no) (fields_autoplaced)
+    (property "Reference" "H2" (at 377.19 64.77 0)
+      (effects (font (size 1.27 1.27)) (justify left))
+    )
+    (property "Value" "Mount" (at 377.19 67.31 0)
+      (effects (font (size 1.27 1.27)) (justify left))
+    )
+    (property "Footprint" "TestPoint:TestPoint_Plated_Hole_D3.0mm" (at 374.65 66.04 0)
+      (effects (font (size 1.27 1.27)) hide)
+    )
+    (property "Datasheet" "~" (at 374.65 66.04 0)
+      (effects (font (size 1.27 1.27)) hide)
+    )
+    (instances
+      (project "80bus"
+        (path "/c5a86bac-f144-45ed-8f39-1fb354fa8f6d"
+          (reference "H2") (unit 1)
+        )
+      )
+    )
+  )
   (symbol (lib_id "Device:R") (at 350.52 233.68 270) (unit 1)
     (in_bom yes) (on_board yes) (dnp no)
@@
         )
       )
+    )
+  )
+  (symbol (lib_id "Mechanical:MountingHole") (at 374.65 78.74 0) (unit 1)
+    (in_bom yes) (on_board yes) (dnp no) (fields_autoplaced)
+    (property "Reference" "H4" (at 377.19 77.47 0)
+      (effects (font (size 1.27 1.27)) (justify left))
+    )
+    (property "Value" "Mount" (at 377.19 80.01 0)
+      (effects (font (size 1.27 1.27)) (justify left))
+    )
+    (property "Footprint" "TestPoint:TestPoint_Plated_Hole_D3.0mm" (at 374.65 78.74 0)
+      (effects (font (size 1.27 1.27)) hide)
+    )
+    (property "Datasheet" "~" (at 374.65 78.74 0)
+      (effects (font (size 1.27 1.27)) hide)
+    )
+    (instances
+      (project "80bus"
+        (path "/c5a86bac-f144-45ed-8f39-1fb354fa8f6d"
+          (reference "H4") (unit 1)
+        )
+      )

Commit message: Docs and Kicad 9
Other:
- title: 80 Bus Compact Flash Card -> 80 Bus Compact Flash Card - Kicad 9
